Commit message: Add ROS Demo

File: ROS/ros_learn/src/urdf_gazebo/urdf/car_full_ver/camera.xacro (robot description, xacro)
@@ -11,5 +11,5 @@
                     <box size="${camera_length} ${camera_width} ${camera_height}" />
                 </geometry>
-                <origin xyz="0 0 0" rpy="0 0 0" />
+                <origin xyz="0 0 0" rpy="0 0 ${PI / 2}" />
                 <material name="laser_support_material">
                     <color rgba="0.3 0.9 0.3 0.9" />
@@ -20,5 +20,5 @@
                     <box size="0.03 0.01 ${camera_height}" />
                 </geometry>
-                <origin xyz="0 0 0" rpy="0 0 0" />
+                <origin xyz="0 0 0" rpy="0 0 ${PI / 2}" />
             </collision>
             <xacro:Box_inertial_matrix m="${camera_mass}" l="${camera_length}" w="${camera_width}"
@@ -30,5 +30,5 @@
             <origin
                 xyz="${base_link_radius - x_offset} 0 ${base_link_length / 2 + camera_height / 2}"
-                rpy="0 0 ${PI / 2}" />
+                rpy="0 0 0" />
         </joint>
         <gazebo reference="camera">

File: ROS/ros_learn/src/urdf_gazebo/urdf/car_full_ver/car_full_ver.xacro (robot description, xacro)
@@ -6,3 +6,4 @@
     <xacro:include filename="laser_sim.xacro"/>
     <xacro:include filename="camera_sim.xacro" />
+    <xacro:include filename="kinetic_sim.xacro" />
 </robot>

File: ROS/ros_learn/src/urdf_gazebo/urdf/car_full_ver/laser.xacro (robot description, xacro)
@@ -53,9 +53,8 @@
             <xacro:cylinder_inertial_matrix m="${laser_mass}" r="${laser_radius}" h="${laser_length}" />
         </link>
-        <joint name="laser_2support_base" type="continuous">
+        <joint name="laser_2support_base" type="fixed">
             <parent link="laser_support"></parent>
             <child link="laser"></child>
             <origin xyz="0 0 ${laser_support_length / 2 + laser_length / 2}" rpy="0 0 0" />
-            <axis xyz="0 0 1" />
         </joint>
         <gazebo reference="laser">
